Commit message: mapping

File: diffrobot_description/urdf/diffrobot.xacro (robot description, xacro)
@@ -194,5 +194,5 @@
         <origin xyz="0.0 0.0 0.0" rpy="0.0 0.0 0.0"/>
         <geometry>
-            <box size="0.1 0.1 0.1"/>
+           <mesh filename="package://diffrobot_description/meshes/kinect sensor.dae"/>
         </geometry>
         <material name="">

Commit message: last_update_(gmaping)

File: diffrobot_description/urdf/diffrobot.xacro (robot description, xacro)
@@ -1,154 +1,167 @@
-<robot xmlns:xacro="http://www.ros.org/wiki/xacro" name="diffrobot">
-<xacro:include filename="$(find diffrobot_description)/urdf/diffrobot.gazebo"/>  /*plugin*/
-<link name="robot_footprint">
-</link>
-<joint name="robot_footprint_joint" type="fixed">
-    <parent link="robot_footprint"/>
-    <child link="base_link"/>
-</joint>
-<link name="base_link">
-    <inertial>
-        <origin xyz="0.0 0.0 0.0" rpy="0.0 0.0 0.0"/>
-        <mass value="5.0"/>
-        <inertia ixx="0.0" ixy="0.0" ixz="0.0" iyy="0.0" iyz="0.0" izz="0.0"/>
-    </inertial>
-    <visual name="base_link_visual">
-        <origin xyz="0.0 0.0 0.0" rpy="0.0 0.0 0.0"/>
-        <geometry>
-            <box size="0.4 0.2 0.1"/>
-        </geometry>
-        <material name="">
+<?xml version='1.0'?>
+<robot name="diffrobot" xmlns:xacro="http://www.ros.org/wiki/xacro">
+    <xacro:include filename="$(find diffrobot_description)/urdf/diffrobot.gazebo"/>
+    <link name="robot_footprint">
+    </link>
+    <joint name="robot_footprint_joint" type="fixed">
+        <parent link="robot_footprint"/>
+        <child link="base_link"/>
+    </joint>
+    <link name="base_link">
+        <inertial>
+            <origin xyz="0.0 0.0 0.0"/>
+            <mass value="20"/>
+            <inertia ixx="0.1" ixy="0.0" ixz="0.0" iyy="0.1" iyz="0.0" izz="0.1"/>
+        </inertial>
+        <visual name='base_link_visual'>
+            <origin xyz="0.0 0.0 0.20" />
+            <geometry>
+                <box size="0.6 0.45 0.1"/>
+            </geometry>
+             <material name="">
             <color rgba="1.0 0.0 0.0 1.0"/>
             <texture filename=""/>
         </material>
-    </visual>
-    <collision>
-        <origin xyz="0.0 0.0 0.0" rpy="0.0 0.0 0.0"/>
-        <geometry>
-            <box size="0.4 0.2 0.1"/>
-        </geometry>
-    </collision>
-</link>
-<link name="left_wheel">
-    <inertial>
-        <origin xyz="0.0 0.0 0.0" rpy="0.0 0.0 0.0"/>
-        <mass value="1.0"/>
-        <inertia ixx="0.0" ixy="0.0" ixz="0.0" iyy="0.0" iyz="0.0" izz="0.0"/>
-    </inertial>
-    <visual name="left_wheel_visual">
-        <origin xyz="0.0 0.0 0.0" rpy="0.0 0.0 0.0"/>
-        <geometry>
-            <cylinder radius="0.1" length="0.05"/>
-        </geometry>
-        <material name="">
-            <color rgba="0.0 1.0 0.0 1.0"/>
-            <texture filename=""/>
-        </material>
-    </visual>
-    <collision>
-        <origin xyz="0.0 0.0 0.0" rpy="0.0 0.0 0.0"/>
-        <geometry>
-            <cylinder radius="0.1" length="0.05"/>
-        </geometry>
-    </collision>
-</link>
-<joint name="left_wheel_joint" type="continuous">
-    <origin xyz="0.0 0.15 0.0" rpy="0.0 1.5705 1.5705"/>
-    <parent link="base_link"/>
-    <child link="left_wheel"/>
-    <axis xyz="0.0 0.0 1.0"/>
-    <limit lower="0.0" upper="0.0" effort="0.0" velocity="0.0"/>
-</joint>
-<link name="right_wheel">
-    <inertial>
-        <origin xyz="0.0 0.0 0.0" rpy="0.0 0.0 0.0"/>
-        <mass value="1.0"/>
-        <inertia ixx="0.0" ixy="0.0" ixz="0.0" iyy="0.0" iyz="0.0" izz="0.0"/>
-    </inertial>
-    <visual name="right_wheel_visual">
-        <origin xyz="0.0 0.0 0.0" rpy="0.0 0.0 0.0"/>
-        <geometry>
-            <cylinder radius="0.1" length="0.05"/>
-        </geometry>
-        <material name="">
-            <color rgba="0.0 1.0 0.0 1.0"/>
-            <texture filename=""/>
-        </material>
-    </visual>
-    <collision>
-        <origin xyz="0.0 0.0 0.0" rpy="0.0 0.0 0.0"/>
-        <geometry>
-            <cylinder radius="0.1" length="0.05"/>
-        </geometry>
-    </collision>
-</link>
-<joint name="right_wheel_joint" type="continuous">
-    <origin xyz="0.0 -0.15 0.0" rpy="0.0 1.5705 1.5705"/>
-    <parent link="base_link"/>
-    <child link="right_wheel"/>
-    <axis xyz="0.0 0.0 1.0"/>
-    <limit lower="0.0" upper="0.0" effort="0.0" velocity="0.0"/>
-</joint>
-<link name="front_caster">
-    <inertial>
-        <origin xyz="0.0 0.0 0.0" rpy="0.0 0.0 0.0"/>
-        <mass value="0.1"/>
-        <inertia ixx="0.0" ixy="0.0" ixz="0.0" iyy="0.0" iyz="0.0" izz="0.0"/>
-    </inertial>
-    <visual name="front_caster_visual">
-        <origin xyz="0.0 0.0 0.0" rpy="0.0 0.0 0.0"/>
-        <geometry>
-            <sphere radius="0.0499"/>
-        </geometry>
-        <material name="">
-            <color rgba="0.0 0.0 1.0 1.0"/>
-            <texture filename=""/>
-        </material>
-    </visual>
-    <collision>
-        <origin xyz="0.0 0.0 0.0" rpy="0.0 0.0 0.0"/>
-        <geometry>
-            <sphere radius="0.0499"/>
-        </geometry>
-    </collision>
-</link>
-    <joint name="front_caster_joint" type="fixed">
-        <origin xyz="0.15 0.0 -0.05" rpy="0.0 0.0 0.0"/>
-        <parent link="base_link"/>
-        <child link="front_caster"/>
-        <axis xyz="0.0 0.0 0.0"/>
-        <limit lower="0.0" upper="0.0" effort="0.0" velocity="0.0"/>
-    </joint>
-<link name="back_caster">
-    <inertial>
-        <origin xyz="0.0 0.0 0.0" rpy="0.0 0.0 0.0"/>
-        <mass value="0.1"/>
-        <inertia ixx="0.0" ixy="0.0" ixz="0.0" iyy="0.0" iyz="0.0" izz="0.0"/>
-    </inertial>
-    <visual name="back_caster_visual">
-        <origin xyz="0.0 0.0 0.0" rpy="0.0 0.0 0.0"/>
-        <geometry>
-            <sphere radius="0.0499"/>
-        </geometry>
-        <material name="">
-            <color rgba="0.0 0.0 1.0 1.0"/>
-            <texture filename=""/>
-        </material>
-    </visual>
-    <collision>
-        <origin xyz="0.0 0.0 0.0" rpy="0.0 0.0 0.0"/>
-        <geometry>
-            <sphere radius="0.0499"/>
-        </geometry>
-    </collision>
-</link>
-    <joint name="back_caster_joint" type="fixed">
-        <origin xyz="-0.15 0.0 -0.05" rpy="0.0 0.0 0.0"/>
-        <parent link="base_link"/>
-        <child link="back_caster"/>
-        <axis xyz="0.0 0.0 0.0"/>
-        <limit lower="0.0" upper="0.0" effort="0.0" velocity="0.0"/>
-    </joint>
-    <link name="lidar_link">
+        </visual>
+        <collision name=''>
+            <origin xyz="0.0 0.0 0.2" rpy="0.0 0.0 0.0"/>
+            <geometry>
+                <box size="0.6 0.45 0.1"/>
+            </geometry>
+        </collision>
+        <visual name='base_link_visual'>
+            <origin xyz="-0.10 0.0 0.30" />
+            <geometry>
+                <box size="0.4 0.45 0.1"/>
+            </geometry>
+             <material name="">
+            <color rgba="1.0 0.0 0.0 1.0"/>
+            <texture filename=""/>
+        </material>
+        </visual>
+        <collision name=''>
+            <origin xyz="-0.10 0.0 0.30" />
+            <geometry>
+                <box size="0.4 0.45 0.1"/>
+            </geometry>
+        </collision>
+        </link>
+    <link name="front_right_wheel">
+    <inertial>
+      <mass value="5"/>
+      <origin rpy="0 0 0" xyz="0 0 0"/>
+      <inertia ixx="0.1" ixy="0" ixz="0" iyy="0.1" iyz="0" izz="0.1"/>
+    </inertial>
+    <collision name="front_right_wheel_collision">
+      <origin rpy="0 1.5707 1.5707" xyz="0 0 0" />
+      <geometry>
+        <cylinder length="0.05" radius="0.1"/>
+      </geometry>
+    </collision>
+    <visual name="front_right_wheel_visual">
+      <origin rpy="0 1.5707 1.5707" xyz="0 0 0"/>
+      <geometry>
+        <cylinder length="0.05" radius="0.1"/>
+      </geometry>
+     <material name="">
+            <color rgba="0.0 1.0 0.0 1.0"/>
+            <texture filename=""/>
+        </material>
+    </visual>
+  </link>
+  <joint name="joint_front_right_wheel" type="continuous">
+    <origin rpy="0 0 0" xyz="0.175 -0.25 0.1"/>
+    <child link="front_right_wheel" />
+    <parent link="base_link"/>
+    <axis rpy="0 0 0" xyz="0 1 0"/>
+  </joint>
+    <link name="front_left_wheel">
+    <inertial>
+      <mass value="5"/>
+      <origin rpy="0 0 0" xyz="0 0 0"/>
+      <inertia ixx="0.1" ixy="0" ixz="0" iyy="0.1" iyz="0" izz="0.1"/>
+    </inertial>
+    <collision name="front_left_wheel_collision">
+      <origin rpy="0 1.5707 1.5707" xyz="0 0 0" />
+      <geometry>
+        <cylinder length="0.05" radius="0.1"/>
+      </geometry>
+    </collision>
+    <visual name="front_left_wheel_visual">
+      <origin rpy="0 1.5707 1.5707" xyz="0 0 0"/>
+      <geometry>
+        <cylinder length="0.05" radius="0.1"/>
+      </geometry>
+      <material name="">
+            <color rgba="0.0 1.0 0.0 1.0"/>
+            <texture filename=""/>
+        </material>
+    </visual>
+  </link>
+  <joint name="joint_front_left_wheel" type="continuous">
+   <origin rpy="0 0 0" xyz="0.175 0.25 0.1"/>
+    <child link="front_left_wheel" />
+    <parent link="base_link"/>
+    <axis rpy="0 0 0" xyz="0 1 0"/>
+  </joint>
+<link name="back_left_wheel">
+    <inertial>
+      <mass value="5"/>
+      <origin rpy="0 0 0" xyz="0 0 0"/>
+      <inertia ixx="0.1" ixy="0" ixz="0" iyy="0.1" iyz="0" izz="0.1"/>
+    </inertial>
+    <collision name="back_left_wheel_collision">
+    <origin xyz="0.0 0.0 0.0" rpy="0.0 0.0 0.0"/>
+      <geometry>
+        <cylinder length="0.05" radius="0.1"/>
+      </geometry>
+    </collision>
+    <visual name="back_left_wheel_visual">
+      <origin xyz="0.0 0.0 0.0" rpy="0.0 0.0 0.0"/>
+      <geometry>
+        <cylinder length="0.05" radius="0.1"/>
+      </geometry>
+      <material name="">
+            <color rgba="0.0 1.0 0.0 1.0"/>
+            <texture filename=""/>
+        </material>
+    </visual>
+  </link>
+  <joint name="joint_back_left_wheel" type="fixed">
+   <origin rpy="0 -1.5707 1.5707" xyz="-0.175 0.25 0.1" />
+    <child link="back_left_wheel" />
+    <parent link="base_link"/>
+    <axis rpy="0 0 0" xyz="0 1 0"/>
+  </joint>
+  <link name="back_right_wheel">
+    <inertial>
+      <mass value="5"/>
+      <origin rpy="0 0 0" xyz="0 0 0"/>
+      <inertia ixx="0.1" ixy="0" ixz="0" iyy="0.1" iyz="0" izz="0.1"/>
+    </inertial>
+    <collision name="back_right_wheel_collision">
+      <origin xyz="0.0 0.0 0.0" rpy="0.0 0.0 0.0"/>
+      <geometry>
+        <cylinder length="0.05" radius="0.1"/>
+      </geometry>
+    </collision>
+    <visual name="back_right_wheel_visual">
+      <origin xyz="0.0 0.0 0.0" rpy="0.0 0.0 0.0"/>
+      <geometry>
+        <cylinder length="0.05" radius="0.1"/>
+      </geometry>
+      <material name="">
+            <color rgba="0.0 1.0 0.0 1.0"/>
+            <texture filename=""/>
+        </material>
+    </visual>
+  </link>
+  <joint name="joint_back_right_wheel" type="fixed">
+    <origin rpy="0 -1.5707 1.5707" xyz="-0.175 -0.25 0.1" />
+    <child link="back_right_wheel" />
+    <parent link="base_link"/>
+    <axis rpy="0 0 0" xyz="0 1 0"/>
+  </joint>
+   <link name="lidar_link">
         <inertial>
             <origin xyz="0.0 0.0 0.0" rpy="0.0 0.0 0.0"/>
@@ -174,5 +187,5 @@
     </link>
     <joint name="lidar_joint" type="fixed">
-         <origin xyz="0.01 0.0 0.12" rpy="1.5708 0.0 1.5708"/>
+         <origin xyz="0.01 0.0 0.39" rpy="1.5708 0.0 1.5708"/>
         <parent link="base_link"/>
         <child link="lidar_link"/>
@@ -185,5 +198,5 @@
     <child link="laser_data_link"/>
 </joint>
-<link name="camera_link">
+   <link name="camera_link">
     <inertial>
         <origin xyz="0.0 0.0 0.0" rpy="0.0 0.0 0.0"/>
@@ -209,5 +222,5 @@
 </link>
 <joint name="camera_joint" type="fixed">
-   <origin xyz="0.17 0.0 0.12" rpy="0.0 0.0 0.0"/>
+   <origin xyz="0.28 0.0 0.30" rpy="0.0 0.0 0.0"/>
     <parent link="base_link"/>
     <child link="camera_link"/>
